File: PCB-KiCad/dbwifi-revB/dbwifi-revB.kicad_pcb (KiCad board)
At the start: 2 copper layers, 29.6 x 40.6 mm, 27 parts, among them J1 [DF13-6P-1.25H], J2 [DF13-6P-1.25H], J3 DF12-4.0-36DP-0.5V, J4 DS1021-1x6S, J5 DS1021-1x6S, U1 TPS76733QD

Commit message: Minor fix in DBWiFi PCB
Routing:
- net +3V3: track 88.0 -> 77.8 mm, vias 13 -> 10
